File: test2.kicad_pcb (KiCad board)
At the start: 2 copper layers, 195.1 x 101.7 mm, 98 parts, among them K1 KEYSW, K10 KEYSW, K11 KEYSW, K12 KEYSW, K13 KEYSW, K14 KEYSW, K15 KEYSW, K16 KEYSW, K17 KEYSW, K18 KEYSW, K19 KEYSW, K2 KEYSW, K20 KEYSW, K21 KEYSW, K22 KEYSW, K23 KEYSW, K24 KEYSW, K25 KEYSW, K26 KEYSW, K27 KEYSW, K28 KEYSW, K29 KEYSW, K3 KEYSW, K30 KEYSW, K31 KEYSW, K32 KEYSW, K33 KEYSW, K34 KEYSW, K35 KEYSW, K36 KEYSW, K37 KEYSW, K38 KEYSW, K39 KEYSW, K4 KEYSW, K40 KEYSW, K5 KEYSW, K6 KEYSW, K7 KEYSW, K8 KEYSW, K9 KEYSW, SW1 SW_PUSH, U1 ProMicro

Commit message: update
Parts:
- moved H1 17.3 mm to (188.2, 74.7)
- moved SW1 13.9 mm to (191.5, 70.1)
- moved U1 11.2 mm to (164.2, 65.9), turned to -15 degrees
Routing:
- net ROW1: track 310.7 -> 328.4 mm
- net GND: track 510.9 -> 526.8 mm
- net COL7: track 101.8 -> 89.4 mm
- net VDD: track 459.8 -> 470.3 mm
- net COL9: track 158.0 -> 147.6 mm
- net COL1: track 161.4 -> 171.4 mm
- net COL8: track 118.3 -> 108.4 mm
- net COL2: track 146.8 -> 155.6 mm
- net COL3: track 142.2 -> 150.1 mm
- net COL4: track 113.2 -> 120.8 mm
- net COL10: track 162.8 -> 155.8 mm
- net COL5: track 97.8 -> 104.0 mm
- net LED: track 157.3 -> 152.4 mm
- net ROW3: track 350.9 -> 354.9 mm
- net ROW2: track 331.8 -> 335.5 mm
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Other:
- board size 195.1 x 101.7 mm -> 195.1 x 106.4 mm
- board text added: "RSLATE"
- board text removed: "Minni Keyboard"
