File: _autosave-V4.kicad_pcb (KiCad board)
At the start: 2 copper layers, 195.1 x 107.9 mm, 98 parts, among them K1 KEYSW, K10 KEYSW, K11 KEYSW, K12 KEYSW, K13 KEYSW, K14 KEYSW, K15 KEYSW, K16 KEYSW, K17 KEYSW, K18 KEYSW, K19 KEYSW, K2 KEYSW, K20 KEYSW, K21 KEYSW, K22 KEYSW, K23 KEYSW, K24 KEYSW, K25 KEYSW, K26 KEYSW, K27 KEYSW, K28 KEYSW, K29 KEYSW, K3 KEYSW, K30 KEYSW, K31 KEYSW, K32 KEYSW, K33 KEYSW, K34 KEYSW, K35 KEYSW, K36 KEYSW, K37 KEYSW, K38 KEYSW, K39 KEYSW, K4 KEYSW, K40 KEYSW, K5 KEYSW, K6 KEYSW, K7 KEYSW, K8 KEYSW, K9 KEYSW, SW1 SW_PUSH, U1 ProMicro

Commit message: nice
Changed lines of the file:
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@@
       (drillshape 0)
       (scaleselection 1)
-      (outputdirectory "gerbr/")
+      (outputdirectory "outputs/gerber/")
     )
   )
@@
     (property "Sheetname" "")
     (attr through_hole)
-    (fp_text reference "SW1" (at 3.25 -2) (layer "F.SilkS")
+    (fp_text reference "SW1" (at 3.25 2.25) (layer "F.SilkS")
       (effects (font (size 1 1) (thickness 0.15)))
     )
