File: V4.kicad_pcb (KiCad board)
At the start: 2 copper layers, 195.1 x 107.9 mm, 98 parts, among them K1 KEYSW, K10 KEYSW, K11 KEYSW, K12 KEYSW, K13 KEYSW, K14 KEYSW, K15 KEYSW, K16 KEYSW, K17 KEYSW, K18 KEYSW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

Commit message: nice
Routing:
- net COL10: track 163.1 -> 162.5 mm
Other:
- board text added: "JLCJLCJLCJLC"
