File: plate/plate.kicad_pcb (KiCad board)
At the start: 2 copper layers, 195.1 x 99.7 mm, 40 parts, among them K1 KEYSW, K10 KEYSW, K11 KEYSW, K12 KEYSW, K13 KEYSW, K14 KEYSW, K15 KEYSW, K16 KEYSW, K17 KEYSW, K18 KEYSW, K19 KEYSW, K2 KEYSW, K20 KEYSW, K21 KEYSW, K22 KEYSW, K23 KEYSW, K24 KEYSW, K25 KEYSW, K26 KEYSW, K27 KEYSW, K28 KEYSW, K29 KEYSW, K3 KEYSW, K30 KEYSW, K31 KEYSW, K32 KEYSW, K33 KEYSW, K34 KEYSW, K35 KEYSW, K36 KEYSW, K37 KEYSW, K38 KEYSW, K39 KEYSW, K4 KEYSW, K40 KEYSW, K5 KEYSW, K6 KEYSW, K7 KEYSW, K8 KEYSW, K9 KEYSW

Commit message: nice
Other:
- board size 195.1 x 99.7 mm -> 195.1 x 99.3 mm
Changed lines of the file:
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@@
   (setup
     (pad_to_mask_clearance 0)
+    (aux_axis_origin 123.7488 32.5374)
     (pcbplotparams
-      (layerselection 0x00010fc_ffffffff)
+      (layerselection 0x0001200_7ffffffe)
       (disableapertmacros false)
       (usegerberextensions false)
@@
       (hpglpendiameter 15.000000)
       (dxfpolygonmode true)
-      (dxfimperialunits true)
+      (dxfimperialunits false)
       (dxfusepcbnewfont true)
       (psnegative false)
@@
       (sketchpadsonfab false)
       (subtractmaskfromsilk false)
-      (outputformat 1)
+      (outputformat 3)
       (mirror false)
-      (drillshape 1)
+      (drillshape 0)
       (scaleselection 1)
       (outputdirectory "")
@@
     (fp_line (start 7 -7) (end 7 7) (layer "Edge.Cuts") (width 0.12))
   )
-  (gr_circle (center 130.7973 59.6265) (end 133.1214 59.6265) (layer "Cmts.User") (width 0.05) (fill none))
   (gr_line (start 135.31364 35.289473) (end 142.035669 37.094871) (layer "Cmts.User") (width 0.05))
   (gr_arc (start 133.44713 36.367102) (mid 134.157201 35.441721) (end 135.31364 35.289473) (layer "Cmts.User") (width 0.05))
-  (gr_circle (center 168.8211 48.9204) (end 171.1452 48.9204) (layer "Cmts.User") (width 0.05) (fill none))
   (gr_line (start 142.035669 37.094871) (end 173.8122 45.6438) (layer "Cmts.User") (width 0.05))
   (gr_arc (start 133.44713 36.367102) (mid 134.157201 35.441721) (end 135.31364 35.289473) (layer "Cmts.User") (width 0.05))
-  (gr_circle (center 164.973 59.8551) (end 167.2971 59.8551) (layer "Cmts.User") (width 0.05) (fill none))
+  (gr_circle (center 131.1783 59.4741) (end 132.3213 59.4741) (layer "Cmts.User") (width 0.05) (fill none))
   (gr_line (start 133.44713 36.367102) (end 126.731518 61.21217) (layer "Cmts.User") (width 0.05))
   (gr_line (start 126.5682 61.8363) (end 136.8933 64.597381) (layer "Cmts.User") (width 0.05))
@@
   (gr_line (start 133.44713 36.367102) (end 126.731518 61.21217) (layer "Cmts.User") (width 0.05))
   (gr_line (start 126.5682 61.8363) (end 133.44713 36.367102) (layer "Cmts.User") (width 0.05))
+  (gr_circle (center 166.0398 60.0837) (end 167.1828 60.0837) (layer "Cmts.User") (width 0.05) (fill none))
   (gr_line (start 168.3639 64.5795) (end 173.8122 45.6438) (layer "Cmts.User") (width 0.05))
-  (gr_line (start 165.4683 43.3959) (end 243.64985 64.311444) (layer "Edge.Cuts") (width 0.1))
-  (gr_circle (center 164.973 59.8551) (end 167.2971 59.8551) (layer "Edge.Cuts") (width 0.1) (fill none))
-  (gr_line (start 173.736 50.1777) (end 173.736 57.7215) (layer "Edge.Cuts") (width 0.1))
-  (gr_line (start 160.0581 63.5127) (end 165.4683 43.3959) (layer "Edge.Cuts") (width 0.1))
+  (gr_circle (center 168.9354 49.53) (end 170.0784 49.53) (layer "Cmts.User") (width 0.05) (fill none))
+  (gr_circle (center 166.0398 60.0837) (end 167.1828 60.0837) (layer "Edge.Cuts") (width 0.05) (fill none))
+  (gr_line (start 166.7637 43.7769) (end 243.64985 64.311444) (layer "Edge.Cuts") (width 0.05))
+  (gr_line (start 173.736 50.1777) (end 173.736 57.7215) (layer "Edge.Cuts") (width 0.05))
+  (gr_line (start 161.3535 63.8937) (end 166.7637 43.7769) (layer "Edge.Cuts") (width 0.05))
   (gr_line (start 242.5065 143.1036) (end 52.0065 143.1036) (layer "Edge.Cuts") (width 0.05))
   (gr_arc (start 244.7925 140.8176) (mid 244.122946 142.434046) (end 242.5065 143.1036) (layer "Edge.Cuts") (width 0.05))
-  (gr_circle (center 130.7973 59.6265) (end 133.1214 59.6265) (layer "Edge.Cuts") (width 0.1) (fill none))
-  (gr_circle (center 90.1065 121.7676) (end 91.2495 121.7676) (layer "Edge.Cuts") (width 0.1) (fill none))
+  (gr_circle (center 90.1065 121.7676) (end 91.2495 121.7676) (layer "Edge.Cuts") (width 0.05) (fill none))
   (gr_line (start 49.7205 140.8176) (end 49.7205 64.6176) (layer "Edge.Cuts") (width 0.05))
-  (gr_circle (center 90.1065 83.6676) (end 91.2495 83.6676) (layer "Edge.Cuts") (width 0.1) (fill none))
-  (gr_circle (center 147.2565 102.7176) (end 148.3995 102.7176) (layer "Edge.Cuts") (width 0.1) (fill none))
-  (gr_line (start 183.2991 50.1777) (end 173.736 50.1777) (layer "Edge.Cuts") (width 0.1))
-  (gr_line (start 183.2991 57.7215) (end 183.2991 50.1777) (layer "Edge.Cuts") (width 0.1))
-  (gr_circle (center 168.8211 48.9204) (end 171.1452 48.9204) (layer "Edge.Cuts") (width 0.1) (fill none))
+  (gr_circle (center 90.1065 83.6676) (end 91.2495 83.6676) (layer "Edge.Cuts") (width 0.05) (fill none))
+  (gr_circle (center 147.2565 102.7176) (end 148.3995 102.7176) (layer "Edge.Cuts") (width 0.05) (fill none))
+  (gr_circle (center 168.9354 49.53) (end 170.0784 49.53) (layer "Edge.Cuts") (width 0.05) (fill none))
+  (gr_line (start 183.2991 50.1777) (end 173.736 50.1777) (layer "Edge.Cuts") (width 0.05))
+  (gr_line (start 183.2991 57.7215) (end 183.2991 50.1777) (layer "Edge.Cuts") (width 0.05))
+  (gr_line (start 160.0581 63.4746) (end 161.3535 63.8937) (layer "Edge.Cuts") (width 0.05))
+  (gr_circle (center 131.1783 59.4741) (end 132.3213 59.4741) (layer "Edge.Cuts") (width 0.05) (fill none))
   (gr_line (start 52.0065 62.3316) (end 51.2445 62.3316) (layer "Edge.Cuts") (width 0.05))
-  (gr_circle (center 204.4065 121.7676) (end 205.5495 121.7676) (layer "Edge.Cuts") (width 0.1) (fill none))
+  (gr_circle (center 204.4065 121.7676) (end 205.5495 121.7676) (layer "Edge.Cuts") (width 0.05) (fill none))
   (gr_arc (start 243.64985 64.311444) (mid 244.47704 64.858493) (end 244.792499 65.7987) (layer "Edge.Cuts") (width 0.05))
   (gr_line (start 49.7205 63.8556) (end 49.7205 64.6176) (layer "Edge.Cuts") (width 0.05))
   (gr_line (start 121.4628 62.3316) (end 125.2347 62.3316) (layer "Edge.Cuts") (width 0.05))
-  (gr_line (start 160.0581 63.4746) (end 128.4351 54.9783) (layer "Edge.Cuts") (width 0.1))
+  (gr_line (start 160.0581 63.4746) (end 128.4351 54.9783) (layer "Edge.Cuts") (width 0.05))
   (gr_arc (start 126.718819 61.202041) (mid 126.1745 62.016668) (end 125.24675 62.3316) (layer "Edge.Cuts") (width 0.05))
   (gr_arc (start 49.7205 63.8556) (mid 50.166869 62.777969) (end 51.2445 62.3316) (layer "Edge.Cuts") (width 0.05))
-  (gr_line (start 126.718819 61.202041) (end 128.4351 54.9783) (layer "Edge.Cuts") (width 0.1))
+  (gr_line (start 126.718819 61.202041) (end 128.4351 54.9783) (layer "Edge.Cuts") (width 0.05))
   (gr_line (start 244.792499 65.7987) (end 244.7925 140.8176) (layer "Edge.Cuts") (width 0.05))
   (gr_line (start 52.0065 62.3316) (end 121.4628 62.3316) (layer "Edge.Cuts") (width 0.05))
-  (gr_circle (center 204.4065 83.6676) (end 205.5495 83.6676) (layer "Edge.Cuts") (width 0.1) (fill none))
-  (gr_line (start 173.736 57.7215) (end 183.2991 57.7215) (layer "Edge.Cuts") (width 0.1))
-  (gr_circle (center 178.4985 60.8076) (end 179.6415 60.8076) (layer "Edge.Cuts") (width 0.1) (fill none))
+  (gr_circle (center 204.4065 83.6676) (end 205.5495 83.6676) (layer "Edge.Cuts") (width 0.05) (fill none))
+  (gr_line (start 173.736 57.7215) (end 183.2991 57.7215) (layer "Edge.Cuts") (width 0.05))
+  (gr_circle (center 178.4985 60.8076) (end 179.6415 60.8076) (layer "Edge.Cuts") (width 0.05) (fill none))
   (gr_arc (start 52.0065 143.1036) (mid 50.390054 142.434046) (end 49.7205 140.8176) (layer "Edge.Cuts") (width 0.05))
 )
